Commit message: new orientations arms

File: my_assets/urdf/origin_v10_arms.urdf (robot description, URDF)
Before this commit: robot avular_origin_v10, 9 links, 8 joints
Joints:
- joint left_front_passive_arm_left_front_wheel_joint: origin xyz=0.15 0 0 rpy=0 1.5708 0 -> xyz=0 0 -0.25 rpy=0 0 0
- joint left_rear_passive_arm_left_rear_wheel_joint: origin xyz=0.15 0 0 rpy=0 1.5708 0 -> xyz=0 0 -0.25 rpy=0 0 0
- joint main_body_left_front_passive_arm_joint: origin xyz=0.205 0.25 0.056 rpy=0 0 1.5708 -> xyz=0.205 0.25 0.056 rpy=-0.5236 0 0
- joint main_body_left_rear_passive_arm_joint: origin xyz=-0.205 0.25 0.056 rpy=0 0 1.5708 -> xyz=-0.205 0.25 0.056 rpy=0.5236 0 0
- joint main_body_right_front_passive_arm_joint: axis 0 -1 0 -> 0 1 0; origin xyz=0.205 -0.25 0.056 rpy=0 0 -1.5708 -> xyz=0.205 -0.25 0.056 rpy=-0.5236 0 0
- joint main_body_right_rear_passive_arm_joint: axis 0 -1 0 -> 0 1 0; origin xyz=-0.205 -0.25 0.056 rpy=0 0 -1.5708 -> xyz=-0.205 -0.25 0.056 rpy=0.5236 0 0
- joint right_front_passive_arm_right_front_wheel_joint: origin xyz=0.15 0 0 rpy=0 1.5708 0 -> xyz=0 0 -0.25 rpy=0 0 0
- joint right_rear_passive_arm_right_rear_wheel_joint: origin xyz=0.15 0 0 rpy=0 1.5708 0 -> xyz=0 0 -0.25 rpy=0 0 0

Commit message: new def

File: my_assets/urdf/origin_v10_arms.urdf (robot description, URDF)
Before this commit: robot avular_origin_v10, 9 links, 8 joints
Joints:
- joint left_front_passive_arm_left_front_wheel_joint: origin xyz=0 0 -0.25 rpy=0 0 0 -> xyz=0 0 -0.3 rpy=0 0 0
- joint left_rear_passive_arm_left_rear_wheel_joint: origin xyz=0 0 -0.25 rpy=0 0 0 -> xyz=0 0 -0.3 rpy=0 0 0
- joint main_body_left_front_passive_arm_joint: origin xyz=0.205 0.25 0.056 rpy=-0.5236 0 0 -> xyz=0.205 0.25 0.056 rpy=0 0 0
- joint main_body_left_rear_passive_arm_joint: origin xyz=-0.205 0.25 0.056 rpy=0.5236 0 0 -> xyz=-0.205 0.25 0.056 rpy=0 0 0
- joint main_body_right_front_passive_arm_joint: origin xyz=0.205 -0.25 0.056 rpy=-0.5236 0 0 -> xyz=0.205 -0.25 0.056 rpy=0 0 0
- joint main_body_right_rear_passive_arm_joint: origin xyz=-0.205 -0.25 0.056 rpy=0.5236 0 0 -> xyz=-0.205 -0.25 0.056 rpy=0 0 0
- joint right_front_passive_arm_right_front_wheel_joint: origin xyz=0 0 -0.25 rpy=0 0 0 -> xyz=0 0 -0.3 rpy=0 0 0
- joint right_rear_passive_arm_right_rear_wheel_joint: origin xyz=0 0 -0.25 rpy=0 0 0 -> xyz=0 0 -0.3 rpy=0 0 0

Commit message: new

File: my_assets/urdf/origin_v10_arms.urdf (robot description, URDF)
Before this commit: robot avular_origin_v10, 9 links, 8 joints
Joints:
- joint main_body_left_front_passive_arm_joint: origin xyz=0.205 0.25 0.056 rpy=0 0 0 -> xyz=0.205 0.25 0.1 rpy=0 0 0
- joint main_body_left_rear_passive_arm_joint: origin xyz=-0.205 0.25 0.056 rpy=0 0 0 -> xyz=-0.205 0.25 0.1 rpy=0 0 0
- joint main_body_right_front_passive_arm_joint: origin xyz=0.205 -0.25 0.056 rpy=0 0 0 -> xyz=0.205 -0.25 0.1 rpy=0 0 0
- joint main_body_right_rear_passive_arm_joint: origin xyz=-0.205 -0.25 0.056 rpy=0 0 0 -> xyz=-0.205 -0.25 0.1 rpy=0 0 0

Commit message: old

File: my_assets/urdf/origin_v10_arms.urdf (robot description, URDF)
Before this commit: robot avular_origin_v10, 9 links, 8 joints
Joints:
- joint left_front_passive_arm_left_front_wheel_joint: origin xyz=0 0 -0.3 rpy=0 0 0 -> xyz=0.15 0 0 rpy=0 1.5708 0
- joint left_rear_passive_arm_left_rear_wheel_joint: origin xyz=0 0 -0.3 rpy=0 0 0 -> xyz=0.15 0 0 rpy=0 1.5708 0
- joint main_body_left_front_passive_arm_joint: origin xyz=0.205 0.25 0.1 rpy=0 0 0 -> xyz=0.205 0.25 0.056 rpy=0 0 1.5708
- joint main_body_left_rear_passive_arm_joint: origin xyz=-0.205 0.25 0.1 rpy=0 0 0 -> xyz=-0.205 0.25 0.056 rpy=0 0 1.5708
- joint main_body_right_front_passive_arm_joint: axis 0 1 0 -> 0 -1 0; origin xyz=0.205 -0.25 0.1 rpy=0 0 0 -> xyz=0.205 -0.25 0.056 rpy=0 0 -1.5708
- joint main_body_right_rear_passive_arm_joint: axis 0 1 0 -> 0 -1 0; origin xyz=-0.205 -0.25 0.1 rpy=0 0 0 -> xyz=-0.205 -0.25 0.056 rpy=0 0 -1.5708
- joint right_front_passive_arm_right_front_wheel_joint: origin xyz=0 0 -0.3 rpy=0 0 0 -> xyz=0.15 0 0 rpy=0 1.5708 0
- joint right_rear_passive_arm_right_rear_wheel_joint: origin xyz=0 0 -0.3 rpy=0 0 0 -> xyz=0.15 0 0 rpy=0 1.5708 0

Commit message: new

File: my_assets/urdf/origin_v10_arms.urdf (robot description, URDF)
Before this commit: robot avular_origin_v10, 12 links, 11 joints
Joints:
- joint main_body_left_front_passive_arm_joint: origin xyz=0.205 0.2 0.0 rpy=0 0 0 -> xyz=0.205 0.2 0.3175 rpy=0 0 0

Commit message: changes

File: my_assets/urdf/origin_v10_arms.urdf (robot description, URDF)
Before this commit: robot avular_origin_v10, 12 links, 11 joints
Joints:
- joint left_front_passive_arm_left_front_wheel_joint: origin xyz=0 0 -0.2 rpy=-1.5707 0 0 -> xyz=0 0.04 -0.2 rpy=-1.5707 0 0

Commit message: entire body correct?

File: my_assets/urdf/origin_v10_arms.urdf (robot description, URDF)
Before this commit: robot avular_origin_v10, 12 links, 11 joints
Joints:
- joint left_rear_passive_arm_left_rear_wheel_joint: origin xyz=0.15 0 0 rpy=0 1.5708 0 -> xyz=0 0.04 -0.2 rpy=-1.5707 0 0; type revolute -> continuous
- joint main_body_left_rear_passive_arm_joint: origin xyz=-0.205 0.25 0.056 rpy=0 0 1.5708 -> xyz=-0.205 0.2 0.3175 rpy=0 0 0
- joint main_body_right_front_passive_arm_joint: origin xyz=0.205 -0.2 0.0 rpy=0 0 0 -> xyz=0.205 -0.2 0.3175 rpy=0 0 0
- joint main_body_right_rear_passive_arm_joint: origin xyz=-0.205 -0.25 0.056 rpy=0 0 -1.5708 -> xyz=-0.205 -0.2 0.3175 rpy=0 0 0
- joint ouster_platform_joint: origin xyz=0.272 0 0.189 rpy=0 0 0 -> xyz=0.272 0 0.38 rpy=0 0 0
- joint right_front_passive_arm_right_front_wheel_joint: origin xyz=0 0 -0.2 rpy=-1.5707 0 0 -> xyz=0 -0.04 -0.2 rpy=-1.5707 0 0; type revolute -> continuous
- joint right_rear_passive_arm_right_rear_wheel_joint: origin xyz=0.15 0 0 rpy=0 1.5708 0 -> xyz=0 -0.04 -0.2 rpy=-1.5707 0 0; type revolute -> continuous

Commit message: final?

File: my_assets/urdf/origin_v10_arms.urdf (robot description, URDF)
Before this commit: robot avular_origin_v10, 12 links, 11 joints
Links:
- link left_rear_passive_arm: geometry collision box size=0.1 0.04 0.3; visual box size=0.1 0.04 0.3
- link right_rear_passive_arm: geometry collision box size=0.1 0.04 0.3; visual box size=0.1 0.04 0.3
Joints:
- joint realsense_joint: origin xyz=0.32 0.03 0.1 rpy=0 0 0 -> xyz=0.32 0.03 0.3175 rpy=0 0 0
