Commit message: cleaning

File: my_assets/urdf/origin_v11.urdf (robot description, URDF)
Before this commit: robot avular_origin_v10, 8 links, 7 joints
Links:
- link left_front_wheel: geometry collision cylinder length=.07 radius=.2; visual cylinder length=.07 radius=.2
- link left_rear_wheel: geometry collision cylinder length=.07 radius=.2; visual cylinder length=.07 radius=.2
- link right_front_wheel: geometry collision cylinder length=.07 radius=.2; visual cylinder length=.07 radius=.2
- link right_rear_wheel: geometry collision cylinder length=.07 radius=.2; visual cylinder length=.07 radius=.2
