Commit message: urdf checks

File: my_assets/urdf/origin_v11_fixed_arms.urdf (robot description, URDF)
Before this commit: robot avular_origin_v10, 12 links, 11 joints
Links:
- removed link left_front_passive_arm
- removed link left_rear_passive_arm
- removed link right_front_passive_arm
- removed link right_rear_passive_arm
- added link left_front_passive_arm_fixed_v1, mass 1.0; collision box size=0.1 0.04 0.2; visual box size=0.1 0.04 0.2
- added link left_rear_passive_arm_fixed_v1, mass 1.0; collision box size=0.1 0.04 0.2; visual box size=0.1 0.04 0.2
- added link right_front_passive_arm_fixed_v1, mass 1.0; collision box size=0.1 0.04 0.2; visual box size=0.1 0.04 0.2
- added link right_rear_passive_arm_fixed_v1, mass 1.0; collision box size=0.1 0.04 0.2; visual box size=0.1 0.04 0.2
Joints:
- removed joint left_front_passive_arm_left_front_wheel_joint
- removed joint left_rear_passive_arm_left_rear_wheel_joint
- removed joint main_body_left_front_passive_arm_joint
- removed joint main_body_left_rear_passive_arm_joint
- removed joint main_body_right_front_passive_arm_joint
- removed joint main_body_right_rear_passive_arm_joint
- removed joint right_front_passive_arm_right_front_wheel_joint
- removed joint right_rear_passive_arm_right_rear_wheel_joint
- added joint left_front_passive_arm_left_front_wheel_joint_fixed: type continuous, parent left_front_passive_arm_fixed_v1, child left_front_wheel, origin xyz=0 0.04 -0.1 rpy=-1.5707 0 0, axis 0 1 0, limit effort=100000.0 velocity=10
- added joint left_rear_passive_arm_left_rear_wheel_joint_fixed: type continuous, parent left_rear_passive_arm_fixed_v1, child left_rear_wheel, origin xyz=0 0.04 -0.1 rpy=-1.5707 0 0, axis 0 1 0, limit effort=100000.0 velocity=10
- added joint main_body_left_front_passive_arm_joint_fixed: type fixed, parent main_body, child left_front_passive_arm_fixed_v1, origin xyz=0.205 0.2 0.3175 rpy=0 0 0
- added joint main_body_left_rear_passive_arm_joint_fixed: type fixed, parent main_body, child left_rear_passive_arm_fixed_v1, origin xyz=-0.205 0.2 0.3175 rpy=0 0 0
- added joint main_body_right_front_passive_arm_joint_fixed: type fixed, parent main_body, child right_front_passive_arm_fixed_v1, origin xyz=0.205 -0.2 0.3175 rpy=0 0 0
- added joint main_body_right_rear_passive_arm_joint_fixed: type fixed, parent main_body, child right_rear_passive_arm_fixed_v1, origin xyz=-0.205 -0.2 0.3175 rpy=0 0 0
- added joint right_front_passive_arm_right_front_wheel_joint_fixed: type continuous, parent right_front_passive_arm_fixed_v1, child right_front_wheel, origin xyz=0 -0.04 -0.1 rpy=-1.5707 0 0, axis 0 1 0, limit effort=100000.0 velocity=10
- added joint right_rear_passive_arm_right_rear_wheel_joint_fixed: type continuous, parent right_rear_passive_arm_fixed_v1, child right_rear_wheel, origin xyz=0 -0.04 -0.1 rpy=-1.5707 0 0, axis 0 1 0, limit effort=100000.0 velocity=10

Commit message: changes

File: my_assets/urdf/origin_v11_fixed_arms.urdf (robot description, URDF)
Before this commit: robot avular_origin_v10, 12 links, 11 joints
Joints:
- joint left_front_passive_arm_left_front_wheel_joint_fixed: origin xyz=0 0.04 -0.15 rpy=-1.5707 0 0 -> xyz=0 0.04 -0.2 rpy=-1.5707 0 0
- joint left_rear_passive_arm_left_rear_wheel_joint_fixed: origin xyz=0 0.04 -0.15 rpy=-1.5707 0 0 -> xyz=0 0.04 -0.2 rpy=-1.5707 0 0
- joint right_front_passive_arm_right_front_wheel_joint_fixed: origin xyz=0 -0.04 -0.15 rpy=-1.5707 0 0 -> xyz=0 -0.04 -0.2 rpy=-1.5707 0 0
- joint right_rear_passive_arm_right_rear_wheel_joint_fixed: origin xyz=0 -0.04 -0.15 rpy=-1.5707 0 0 -> xyz=0 -0.04 -0.2 rpy=-1.5707 0 0
