Commit message: dimension update

File: my_assets/urdf/origin_v11_arms.urdf (robot description, URDF)
Before this commit: robot avular_origin_v10, 12 links, 11 joints
Joints:
- joint left_front_passive_arm_left_front_wheel_joint: origin xyz=0 0.04 -0.1 rpy=-1.5707 0 0 -> xyz=0 0.04 -0.15 rpy=-1.5707 0 0
- joint left_rear_passive_arm_left_rear_wheel_joint: origin xyz=0 0.04 -0.1 rpy=-1.5707 0 0 -> xyz=0 0.04 -0.15 rpy=-1.5707 0 0
- joint right_front_passive_arm_right_front_wheel_joint: origin xyz=0 -0.04 -0.1 rpy=-1.5707 0 0 -> xyz=0 -0.04 -0.15 rpy=-1.5707 0 0
- joint right_rear_passive_arm_right_rear_wheel_joint: origin xyz=0 -0.04 -0.1 rpy=-1.5707 0 0 -> xyz=0 -0.04 -0.15 rpy=-1.5707 0 0

File: my_assets/urdf/origin_v11_fixed_arms.urdf (robot description, URDF)
Before this commit: robot avular_origin_v10, 12 links, 11 joints
Joints:
- joint left_front_passive_arm_left_front_wheel_joint_fixed: origin xyz=0 0.04 -0.1 rpy=-1.5707 0 0 -> xyz=0 0.04 -0.15 rpy=-1.5707 0 0
- joint left_rear_passive_arm_left_rear_wheel_joint_fixed: origin xyz=0 0.04 -0.1 rpy=-1.5707 0 0 -> xyz=0 0.04 -0.15 rpy=-1.5707 0 0
- joint right_front_passive_arm_right_front_wheel_joint_fixed: origin xyz=0 -0.04 -0.1 rpy=-1.5707 0 0 -> xyz=0 -0.04 -0.15 rpy=-1.5707 0 0
- joint right_rear_passive_arm_right_rear_wheel_joint_fixed: origin xyz=0 -0.04 -0.1 rpy=-1.5707 0 0 -> xyz=0 -0.04 -0.15 rpy=-1.5707 0 0

Commit message: unique namespace

File: my_assets/urdf/origin_v11_arms.urdf (robot description, URDF)
Before this commit: robot avular_origin_v10, 12 links, 11 joints
Links:
- removed link camera_link
- removed link left_front_passive_arm
- removed link left_front_wheel
- removed link left_rear_passive_arm
- removed link left_rear_wheel
- removed link lidar_link_gazebo
- removed link main_body
- removed link ouster_base
- removed link right_front_passive_arm
- removed link right_front_wheel
- removed link right_rear_passive_arm
- removed link right_rear_wheel
- added link camera_link_v11, mass 0.035; collision box size=0.008 0.13 0.022
- added link left_front_passive_arm_v11, mass 1.0; collision box size=0.1 0.04 0.2; visual box size=0.1 0.04 0.2
- added link left_front_wheel_v11, mass 1; collision cylinder length=.07 radius=.1175; visual cylinder length=.07 radius=.1175
- added link left_rear_passive_arm_v11, mass 1.0; collision box size=0.1 0.04 0.2; visual box size=0.1 0.04 0.2
- added link left_rear_wheel_v11, mass 1; collision cylinder length=.07 radius=.1175; visual cylinder length=.07 radius=.1175
- added link lidar_link_gazebo_v11, mass 0.1; collision cylinder length=0.07 radius=0.04
- added link main_body_v11, mass 21.0; collision box size=.65 .4 .125; visual box size=.65 .4 .125
- added link ouster_base_v11, mass 1; collision box size=0.1 0.1 0.1; visual box size=0.1 0.1 0.1
- added link right_front_passive_arm_v11, mass 1.0; collision box size=0.1 0.04 0.2; visual box size=0.1 0.04 0.2
- added link right_front_wheel_v11, mass 1; collision cylinder length=.07 radius=.1175; visual cylinder length=.07 radius=.1175
- added link right_rear_passive_arm_v11, mass 1.0; collision box size=0.1 0.04 0.2; visual box size=0.1 0.04 0.2
- added link right_rear_wheel_v11, mass 1; collision cylinder length=.07 radius=.1175; visual cylinder length=.07 radius=.1175
Joints:
- removed joint left_front_passive_arm_left_front_wheel_joint
- removed joint left_rear_passive_arm_left_rear_wheel_joint
- removed joint lidar_joint_gazebo
- removed joint main_body_left_front_passive_arm_joint
- removed joint main_body_left_rear_passive_arm_joint
- removed joint main_body_right_front_passive_arm_joint
- removed joint main_body_right_rear_passive_arm_joint
- removed joint ouster_platform_joint
- removed joint realsense_joint
- removed joint right_front_passive_arm_right_front_wheel_joint
- removed joint right_rear_passive_arm_right_rear_wheel_joint
- added joint ight_front_wheel_joint_v11: type continuous, parent right_front_passive_arm_v11, child right_front_wheel_v11, origin xyz=0 -0.04 -0.15 rpy=-1.5707 0 0, axis 0 1 0, limit effort=100000.0 velocity=10
- added joint left_front_passive_arm_joint_v11: type revolute, parent main_body_v11, child left_front_passive_arm_v11, origin xyz=0.205 0.2 0.3175 rpy=0 0 0, axis 0 1 0, limit lower=-0.7854 upper=0.0 effort=100000.0 velocity=10
- added joint left_front_wheel_joint_v11: type continuous, parent left_front_passive_arm_v11, child left_front_wheel_v11, origin xyz=0 0.04 -0.15 rpy=-1.5707 0 0, axis 0 1 0, limit effort=100000.0 velocity=10
- added joint left_rear_wheel_joint_v11: type continuous, parent left_rear_passive_arm_v11, child left_rear_wheel_v11, origin xyz=0 0.04 -0.15 rpy=-1.5707 0 0, axis 0 1 0, limit effort=100000.0 velocity=10
- added joint lidar_joint_gazebo_v11: type fixed, parent ouster_base_v11, child lidar_link_gazebo_v11, origin xyz=0 0 0.035 rpy=0 0 0
- added joint ouster_platform_joint_v11: type fixed, parent main_body_v11, child ouster_base_v11, origin xyz=0.272 0 0.38 rpy=0 0 0
- added joint realsense_joint_v11: type fixed, parent main_body_v11, child camera_link_v11, origin xyz=0.32 0.03 0.3175 rpy=0 0 0
- added joint rear_passive_arm_joint_v11: type revolute, parent main_body_v11, child left_rear_passive_arm_v11, origin xyz=-0.205 0.2 0.3175 rpy=0 0 0, axis 0 1 0, limit lower=0.0 upper=0.7854 effort=100000.0 velocity=10
- added joint right_front_passive_arm_joint_v11: type revolute, parent main_body_v11, child right_front_passive_arm_v11, origin xyz=0.205 -0.2 0.3175 rpy=0 0 0, axis 0 -1 0, limit lower=-0.7854 upper=0.0 effort=100000.0 velocity=10
- added joint right_rear_passive_arm_joint_v11: type revolute, parent main_body_v11, child right_rear_passive_arm_v11, origin xyz=-0.205 -0.2 0.3175 rpy=0 0 0, axis 0 -1 0, limit lower=0.0 upper=0.7854 effort=100000.0 velocity=10
- added joint right_rear_wheel_joint_v11: type continuous, parent right_rear_passive_arm_v11, child right_rear_wheel_v11, origin xyz=0 -0.04 -0.15 rpy=-1.5707 0 0, axis 0 1 0, limit effort=100000.0 velocity=10

File: my_assets/urdf/origin_v11_fixed_arms.urdf (robot description, URDF)
Before this commit: robot avular_origin_v10, 12 links, 11 joints
Links:
- removed link camera_link
- removed link left_front_passive_arm_fixed_v1
- removed link left_front_wheel
- removed link left_rear_passive_arm_fixed_v1
- removed link left_rear_wheel
- removed link lidar_link_gazebo
- removed link main_body
- removed link ouster_base
- removed link right_front_passive_arm_fixed_v1
- removed link right_front_wheel
- removed link right_rear_passive_arm_fixed_v1
- removed link right_rear_wheel
- added link camera_link_v11f, mass 0.035; collision box size=0.008 0.13 0.022
- added link left_front_passive_arm_v11f, mass 1.0; collision box size=0.1 0.04 0.2; visual box size=0.1 0.04 0.2
- added link left_front_wheel_v11f, mass 1; collision cylinder length=.07 radius=.1175; visual cylinder length=.07 radius=.1175
- added link left_rear_passive_arm_v11f, mass 1.0; collision box size=0.1 0.04 0.2; visual box size=0.1 0.04 0.2
- added link left_rear_wheel_v11f, mass 1; collision cylinder length=.07 radius=.1175; visual cylinder length=.07 radius=.1175
- added link lidar_link_gazebo_v11f, mass 0.1; collision cylinder length=0.07 radius=0.04
- added link main_body_v11f, mass 21.0; collision box size=.65 .4 .125; visual box size=.65 .4 .125
- added link ouster_base_v11f, mass 1; collision box size=0.1 0.1 0.1; visual box size=0.1 0.1 0.1
- added link right_front_passive_arm_v11f, mass 1.0; collision box size=0.1 0.04 0.2; visual box size=0.1 0.04 0.2
- added link right_front_wheel_v11f, mass 1; collision cylinder length=.07 radius=.1175; visual cylinder length=.07 radius=.1175
- added link right_rear_passive_arm_v11f, mass 1.0; collision box size=0.1 0.04 0.2; visual box size=0.1 0.04 0.2
- added link right_rear_wheel_v11f, mass 1; collision cylinder length=.07 radius=.1175; visual cylinder length=.07 radius=.1175
Joints:
- removed joint left_front_passive_arm_left_front_wheel_joint_fixed
- removed joint left_rear_passive_arm_left_rear_wheel_joint_fixed
- removed joint lidar_joint_gazebo
- removed joint main_body_left_front_passive_arm_joint_fixed
- removed joint main_body_left_rear_passive_arm_joint_fixed
- removed joint main_body_right_front_passive_arm_joint_fixed
- removed joint main_body_right_rear_passive_arm_joint_fixed
- removed joint ouster_platform_joint
- removed joint realsense_joint
- removed joint right_front_passive_arm_right_front_wheel_joint_fixed
- removed joint right_rear_passive_arm_right_rear_wheel_joint_fixed
- added joint left_front_passive_arm_joint_v11f: type fixed, parent main_body_v11f, child left_front_passive_arm_v11f, origin xyz=0.205 0.2 0.3175 rpy=0 0 0
- added joint left_front_wheel_joint_v11f: type continuous, parent left_front_passive_arm_v11f, child left_front_wheel_v11f, origin xyz=0 0.04 -0.2 rpy=-1.5707 0 0, axis 0 1 0, limit effort=100000.0 velocity=10
- added joint left_rear_passive_arm_joint_v11f: type fixed, parent main_body_v11f, child left_rear_passive_arm_v11f, origin xyz=-0.205 0.2 0.3175 rpy=0 0 0
- added joint left_rear_wheel_joint_v11f: type continuous, parent left_rear_passive_arm_v11f, child left_rear_wheel_v11f, origin xyz=0 0.04 -0.2 rpy=-1.5707 0 0, axis 0 1 0, limit effort=100000.0 velocity=10
- added joint lidar_joint_gazebo_v11f: type fixed, parent ouster_base_v11f, child lidar_link_gazebo_v11f, origin xyz=0 0 0.035 rpy=0 0 0
- added joint ouster_platform_joint_v11f: type fixed, parent main_body_v11f, child ouster_base_v11f, origin xyz=0.272 0 0.38 rpy=0 0 0
- added joint realsense_joint_v11f: type fixed, parent main_body_v11f, child camera_link_v11f, origin xyz=0.32 0.03 0.3175 rpy=0 0 0
- added joint right_front_passive_arm_joint_v11f: type fixed, parent main_body_v11f, child right_front_passive_arm_v11f, origin xyz=0.205 -0.2 0.3175 rpy=0 0 0
- added joint right_front_wheel_joint_v11f: type continuous, parent right_front_passive_arm_v11f, child right_front_wheel_v11f, origin xyz=0 -0.04 -0.2 rpy=-1.5707 0 0, axis 0 1 0, limit effort=100000.0 velocity=10
- added joint right_rear_passive_arm_joint_v11f: type fixed, parent main_body_v11f, child right_rear_passive_arm_v11f, origin xyz=-0.205 -0.2 0.3175 rpy=0 0 0
- added joint right_rear_wheel_joint_v11f: type continuous, parent right_rear_passive_arm_v11f, child right_rear_wheel_v11f, origin xyz=0 -0.04 -0.2 rpy=-1.5707 0 0, axis 0 1 0, limit effort=100000.0 velocity=10
