Commit message: start on Option-Critic Agent

File: my_assets/urdf/origin_v10.urdf (robot description, URDF)
Before this commit: robot avular_origin_v10, 11 links, 10 joints
Links:
- link gnss_link: geometry visual box size=0.03 0.03 0.1
- link left_front_wheel: geometry collision cylinder length=.07 radius=.1175; visual cylinder length=.07 radius=.1175
- link left_rear_wheel: geometry collision cylinder length=.07 radius=.1175; visual cylinder length=.07 radius=.1175
- link main_body: geometry collision box size=.65 .4 .125; visual box size=.65 .4 .125
- link ouster_base: geometry collision box size=0.1 0.1 0.1; visual box size=0.1 0.1 0.1
- link right_front_wheel: geometry collision cylinder length=.07 radius=.1175; visual cylinder length=.07 radius=.1175
- link right_rear_wheel: geometry collision cylinder length=.07 radius=.1175; visual cylinder length=.07 radius=.1175

Commit message: urdf final touches

File: my_assets/urdf/origin_v10.urdf (robot description, URDF)
Before this commit: robot avular_origin_v10, 11 links, 10 joints
Links:
- removed link gnss_link
- removed link os_sensor
Joints:
- removed joint gnss_joint
- removed joint ouster_orientation_joint

Commit message: new names

File: my_assets/urdf/origin_v10.urdf (robot description, URDF)
Before this commit: robot avular_origin_v10, 8 links, 7 joints
Joints:
- removed joint main_body_left_front_wheel
- removed joint main_body_left_rear_wheel
- removed joint main_body_right_front_wheel
- removed joint main_body_right_rear_wheel
- added joint eft_rear_wheel_joint: type continuous, parent main_body, child left_rear_wheel, origin xyz=-0.205 0.25 0.056 rpy=-1.5707 0 0, axis 0 0 1, limit effort=100000.0 velocity=10
- added joint left_front_wheel_joint: type continuous, parent main_body, child left_front_wheel, origin xyz=0.205 0.25 0.056 rpy=-1.5707 0 0, axis 0 0 1, limit effort=100000.0 velocity=10
- added joint right_front_wheel_joint: type continuous, parent main_body, child right_front_wheel, origin xyz=0.205 -0.25 0.056 rpy=1.5707 0 0, axis 0 0 -1, limit effort=100000.0 velocity=10
- added joint right_rear_wheel_joint: type continuous, parent main_body, child right_rear_wheel, origin xyz=-0.205 -0.25 0.056 rpy=1.5707 0 0, axis 0 0 -1, limit effort=100000.0 velocity=10
